File: kicad/voltage-sense/voltage-sense.sch (KiCad schematic (older format))
At the start: 4 parts, among them J1 Conn_01x04_Male, Q1 Si4532DY

Commit message: minor fixes
Parts:
- Q1: value Si4532DY -> Si9942DY
Connections:
- net 3.68V: now reaches Q1.4 (G), Q1.7 (D), Q1.8 (D), R1.2
Other:
- note added: "drain\n"
- note added: "source"
Changed lines of the file:
@@
 P 4500 2550
 F 0 "Q1" H 4705 2596 50  0000 L CNN
-F 1 "Si4532DY" H 4705 2505 50  0000 L CNN
+F 1 "Si9942DY" H 4705 2505 50  0000 L CNN
 F 2 "Package_SO:SOIC-8_3.9x4.9mm_P1.27mm" H 4700 2475 50  0001 L CNN
 F 3 "https://www.onsemi.com/pub/Collateral/SI4532DY-D.PDF" H 4600 2550 50  0001 L CNN
@@
 P 3950 3200
 F 0 "Q1" H 4155 3246 50  0000 L CNN
-F 1 "Si4532DY" H 4155 3155 50  0000 L CNN
+F 1 "Si9942DY" H 4155 3155 50  0000 L CNN
 F 2 "Package_SO:SOIC-8_3.9x4.9mm_P1.27mm" H 4150 3125 50  0001 L CNN
 F 3 "https://www.onsemi.com/pub/Collateral/SI4532DY-D.PDF" H 4050 3200 50  0001 L CNN
@@
 Wire Wire Line
 	4050 3500 4050 3700
+Text Label 4650 2050 0    50   ~ 10
+4.11V
+Text Label 4050 3000 0    50   ~ 10
+3.68V
+Text Label 3550 3150 0    50   ~ 10
+0V
+Text Label 4100 3500 0    50   ~ 10
+0V
+Text Notes 4650 2400 0    50   ~ 0
+source
+Text Notes 4650 2750 0    50   ~ 0
+drain\n
+Text Notes 4100 3100 0    50   ~ 0
+drain\n
+Text Notes 4100 3350 0    50   ~ 0
+source
 $EndSCHEMATC
